File: KiCAD/KnurCAN_V2/KnurCAN_V2.kicad_pcb (KiCad board)
At the start: 2 copper layers, 55 x 34 mm, 23 parts, among them J1 Conn_01x07, J2 Conn_01x05, K1 COMUS_3572.1220.X4, Q1 2N7000, Q2 BC547, Q3 BS250, U1 LONGAN_I2C_CAN, U2 LM2903

Commit message: design file updates
Parts:
- moved Q3 5.09 mm to (59.1, 71.9), turned to -90 degrees
Connections:
- Q3 pad 1: VCC_CAN -> 5V
- Q3 pad 3: 5V -> VCC_CAN
Routing:
- net SDA: track 21.8 -> 22.4 mm
Changed lines of the file:
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@@
 			(psa4output no)
 			(plot_black_and_white yes)
-			(plotinvisibletext no)
 			(sketchpadsonfab no)
 			(plotpadnumbers no)
@@
 			)
 		)
-		(property "Datasheet" ""
+		(property "Datasheet" "~"
 			(at 0 0 0)
 			(unlocked yes)
@@
 			)
 		)
-		(property "Datasheet" ""
+		(property "Datasheet" "~"
 			(at 0 0 0)
 			(unlocked yes)
@@
 	(footprint "Package_TO_SOT_THT:TO-92_Inline_Wide"
 		(layer "F.Cu")
-		(at 59.563 76.962 90)
+		(at 59.094 71.896 -90)
 		(descr "TO-92 leads in-line, wide, drill 0.75mm (see NXP sot054_po.pdf)")
 		(tags "to-92 sc-43 sc-43a sot54 PA33 transistor")
 		(property "Reference" "Q3"
-			(at 2.54 -1.397 270)
+			(at 2.54 -1.397 90)
 			(layer "F.SilkS")
 			(effects
@@
 		)
 		(property "Datasheet" "http://www.vishay.com/docs/70209/70209.pdf"
-			(at 0 0 90)
+			(at 0 0 270)
 			(unlocked yes)
 			(layer "F.Fab")
@@
 		)
 		(property "Description" "-0.18A Id, -45V Vds, P-Channel MOSFET, TO-92"
-			(at 0 0 90)
+			(at 0 0 270)
 			(unlocked yes)
 			(layer "F.Fab")
@@
 		)
 		(fp_arc
-			(start 2.54 -2.6)
-			(mid 3.936979 -2.192818)
-			(end 4.8964 -1.098807)
+			(start 0.74 1.85)
+			(mid 0.446097 1.509328)
+			(end 0.215816 1.122795)
 			(stroke
 				(width 0.12)
@@
 		)
 		(fp_arc
-			(start 0.1836 -1.098807)
-			(mid 1.143021 -2.192817)
-			(end 2.54 -2.6)
+			(start 4.864184 1.122795)
+			(mid 4.633903 1.509328)
+			(end 4.34 1.85)
 			(stroke
 				(width 0.12)
@@
 		)
 		(fp_arc
-			(start 4.864184 1.122795)
-			(mid 4.633903 1.509328)
-			(end 4.34 1.85)
+			(start 0.1836 -1.098807)
+			(mid 1.143021 -2.192817)
+			(end 2.54 -2.6)
 			(stroke
 				(width 0.12)
@@
 		)
 		(fp_arc
-			(start 0.74 1.85)
-			(mid 0.446097 1.509328)
-			(end 0.215816 1.122795)
+			(start 2.54 -2.6)
+			(mid 3.936979 -2.192818)
+			(end 4.8964 -1.098807)
 			(stroke
 				(width 0.12)
@@
 		)
 		(fp_line
-			(start -1.01 -2.73)
-			(end 6.09 -2.73)
+			(start 6.09 2.01)
+			(end -1.01 2.01)
 			(stroke
 				(width 0.05)
@@
 		)
 		(fp_line
-			(start -1.01 -2.73)
-			(end -1.01 2.01)
+			(start 6.09 2.01)
+			(end 6.09 -2.73)
 			(stroke
 				(width 0.05)
@@
 		)
 		(fp_line
-			(start 6.09 2.01)
-			(end 6.09 -2.73)
+			(start -1.01 -2.73)
+			(end -1.01 2.01)
 			(stroke
 				(width 0.05)
@@
 		)
 		(fp_line
-			(start 6.09 2.01)
-			(end -1.01 2.01)
+			(start -1.01 -2.73)
+			(end 6.09 -2.73)
 			(stroke
 				(width 0.05)
@@
 		)
 		(fp_arc
-			(start 2.54 -2.48)
-			(mid 4.831221 -0.949055)
-			(end 4.293625 1.753625)
+			(start 0.786375 1.753625)
+			(mid 0.248779 -0.949055)
+			(end 2.54 -2.48)
 			(stroke
 				(width 0.1)
@@
 		)
 		(fp_arc
-			(start 0.786375 1.753625)
-			(mid 0.248779 -0.949055)
-			(end 2.54 -2.48)
+			(start 2.54 -2.48)
+			(mid 4.831221 -0.949055)
+			(end 4.293625 1.753625)
 			(stroke
 				(width 0.1)
@@
 		)
 		(pad "1" thru_hole rect
-			(at 0 0 90)
+			(at 0 0 270)
 			(size 1.5 1.5)
 			(drill 0.8)
 			(layers "*.Cu" "*.Mask")
 			(remove_unused_layers no)
-			(net 18 "VCC_CAN")
-			(pinfunction "D")
+			(net 1 "5V")
+			(pinfunction "S")
 			(pintype "passive")
 		)
 		(pad "2" thru_hole circle
-			(at 2.54 0 90)
+			(at 2.54 0 270)
 			(size 1.5 1.5)
 			(drill 0.8)
@@
 		)
 		(pad "3" thru_hole circle
-			(at 5.08 0 90)
+			(at 5.08 0 270)
 			(size 1.5 1.5)
 			(drill 0.8)
 			(layers "*.Cu" "*.Mask")
 			(remove_unused_layers no)
-			(net 1 "5V")
-			(pinfunction "S")
+			(net 18 "VCC_CAN")
+			(pinfunction "D")
 			(pintype "passive")
 		)
@@
 			)
 		)
-		(property "Datasheet" ""
+		(property "Datasheet" "~"
 			(at 0 0 90)
 			(unlocked yes)
@@
 			)
 		)
-		(property "Datasheet" ""
+		(property "Datasheet" "~"
 			(at 0 0 180)
 			(unlocked yes)
@@
 			)
 		)
-		(property "Datasheet" ""
+		(property "Datasheet" "~"
 			(at 0 0 90)
 			(unlocked yes)
@@
 			)
 		)
-		(property "Datasheet" ""
+		(property "Datasheet" "~"
 			(at 0 0 270)
 			(unlocked yes)
@@
 			)
 		)
-		(property "Datasheet" ""
+		(property "Datasheet" "~"
 			(at 0 0 90)
 			(unlocked yes)
@@
 			)
 		)
-		(property "Datasheet" ""
+		(property "Datasheet" "~"
 			(at 0 0 0)
 			(unlocked yes)
@@
 			)
 		)
-		(property "Datasheet" ""
+		(property "Datasheet" "~"
 			(at 0 0 270)
 			(unlocked yes)
@@
 			)
 		)
-		(property "Datasheet" ""
+		(property "Datasheet" "~"
 			(at 0 0 90)
 			(unlocked yes)
@@
 			)
 		)
-		(property "Datasheet" ""
+		(property "Datasheet" "~"
 			(at 0 0 180)
 			(unlocked yes)
@@
 			)
 		)
-		(property "Datasheet" ""
+		(property "Datasheet" "~"
 			(at 0 0 90)
 			(unlocked yes)
@@
 			)
 		)
-		(property "Datasheet" ""
+		(property "Datasheet" "~"
 			(at 0 0 180)
 			(unlocked yes)
@@
 			)
 		)
-		(property "Datasheet" ""
+		(property "Datasheet" "~"
 			(at 0 0 90)
 			(unlocked yes)
@@
 			)
 		)
-		(property "Datasheet" ""
+		(property "Datasheet" "~"
 			(at 0 0 0)
 			(unlocked yes)
@@
 	)
 	(segment
+		(start 54.61 84.582)
+		(end 56.943056 82.248944)
+		(width 0.762)
+		(layer "B.Cu")
+		(net 1)
+	)
+	(segment
 		(start 97.77 89.528)
 		(end 97.382 89.916)
@@
 	)
 	(segment
+		(start 56.943056 82.248944)
+		(end 56.943056 74.046944)
+		(width 0.762)
+		(layer "B.Cu")
+		(net 1)
+	)
+	(segment
 		(start 91.313 81.153)
 		(end 91.313 84.201)
@@
 	)
 	(segment
-		(start 56.943056 74.501944)
-		(end 59.563 71.882)
+		(start 56.943056 74.046944)
+		(end 59.094 71.896)
 		(width 0.762)
 		(layer "B.Cu")
@@
 	)
 	(segment
-		(start 54.61 84.582)
-		(end 56.943056 82.248944)
+		(start 59.108 71.882)
+		(end 59.094 71.896)
 		(width 0.762)
 		(layer "B.Cu")
@@
 	)
 	(segment
-		(start 59.161 71.882)
-		(end 63.373 71.882)
+		(start 63.373 71.882)
+		(end 59.108 71.882)
 		(width 0.762)
 		(layer "B.Cu")
@@
 	)
 	(segment
-		(start 56.943056 82.248944)
-		(end 56.943056 74.501944)
-		(width 0.762)
-		(layer "B.Cu")
-		(net 1)
-	)
-	(segment
 		(start 89.96663 85.94)
 		(end 87.122 88.78463)
@@
 	)
 	(segment
-		(start 55.245 72.39)
-		(end 58.547 75.692)
+		(start 57.926 75.706)
+		(end 62.146 75.706)
 		(width 0.508)
 		(layer "F.Cu")
@@
 	)
 	(segment
-		(start 54.61 72.39)
-		(end 55.245 72.39)
+		(start 66.18 79.74)
+		(end 66.33 79.74)
 		(width 0.508)
 		(layer "F.Cu")
@@
 	)
 	(segment
-		(start 58.547 75.692)
-		(end 62.132 75.692)
+		(start 62.146 75.706)
+		(end 66.18 79.74)
 		(width 0.508)
 		(layer "F.Cu")
@@
 	)
 	(segment
-		(start 66.18 79.74)
-		(end 66.33 79.74)
+		(start 54.61 72.39)
+		(end 55.245 72.39)
 		(width 0.508)
 		(layer "F.Cu")
@@
 	)
 	(segment
-		(start 62.132 75.692)
-		(end 66.18 79.74)
+		(start 54.61 72.39)
+		(end 57.926 75.706)
 		(width 0.508)
 		(layer "F.Cu")
@@
 	)
 	(segment
-		(start 60.071 76.962)
-		(end 60.849 77.74)
-		(width 0.508)
-		(layer "B.Cu")
-		(net 18)
-	)
-	(segment
-		(start 59.161 76.962)
-		(end 60.071 76.962)
+		(start 66.33 77.74)
+		(end 59.858 77.74)
 		(width 0.508)
 		(layer "B.Cu")
@@
 	)
 	(segment
-		(start 60.849 77.74)
-		(end 66.33 77.74)
+		(start 59.858 77.74)
+		(end 59.094 76.976)
 		(width 0.508)
 		(layer "B.Cu")
@@
 	)
 	(segment
-		(start 62.865 80.01)
-		(end 63.373 79.502)
+		(start 59.055 80.01)
+		(end 57.835 78.79)
 		(width 0.508)
 		(layer "B.Cu")
@@
 	)
 	(segment
-		(start 58.304 75.681)
-		(end 59.563 74.422)
+		(start 57.835 75.695)
+		(end 59.094 74.436)
 		(width 0.508)
 		(layer "B.Cu")
@@
 	)
 	(segment
-		(start 59.055 80.01)
-		(end 58.304 79.259)
+		(start 62.865 80.01)
+		(end 63.373 79.502)
 		(width 0.508)
 		(layer "B.Cu")
@@
 	)
 	(segment
-		(start 58.304 79.259)
-		(end 58.304 75.681)
+		(start 57.835 78.79)
+		(end 57.835 75.695)
 		(width 0.508)
 		(layer "B.Cu")
