File: KiCAD/KnurCAN_V2/KnurCAN_V2.kicad_sch (KiCad schematic)
At the start: 23 parts, among them J1 Conn_01x07, J2 Conn_01x05, K1 COMUS_3572.1220.X4, Q1 2N7000, Q2 BC547, Q3 BS250, U1 LONGAN_I2C_CAN, U2 LM2903

Commit message: design file updates
Connections:
- net 5V: now also Q3.1 (S); no longer Q3.3 (S)
- net VCC_CAN: now also Q3.3 (D); no longer Q3.1 (D)
